File: Hardware/Qwiic Solid State Relay.brd (EAGLE design)
At the start: 90.2 x 67.3 mm, 73 parts, among them J2 Qwiic Right Angle, J3 Qwiic Right Angle, J9 AVR_SPI_PROG_3X2TESTPOINTS, K1 25A Solid State Relay, K2 25A Solid State Relay, Q1 600mA/40V, Q2 600mA/40V, U4 ATTINY84-ARDUINO

Commit message: flipping relay footprint
Parts:
- moved J4 17.8 mm to (14.0, 59.1), turned to 180 degrees
- moved J5 17.8 mm to (58.4, 59.1), turned to 180 degrees
- moved U$8 17.8 mm to (64.6, 62.2)
- moved U$7 17.8 mm to (20.2, 62.2)
- moved R8 14.0 mm to (74.9, 55.9)
- moved LOGO3 14.0 mm to (40.1, 53.3)
- moved U$2 14.0 mm to (60.7, 47.0)
- moved U$3 14.0 mm to (60.8, 40.6)
- moved D3 11.4 mm to (27.9, 61.0)
- moved D4 11.4 mm to (72.4, 61.0)
- moved R7 11.4 mm to (27.9, 55.9)
- moved U$10 11.4 mm to (72.0, 61.0)
- moved U$9 11.4 mm to (27.9, 61.0)
- turned R5 to 270 degrees
Routing:
- net N$3: track 25.7 -> 19.9 mm
- net N$10: track 21.9 -> 18.5 mm
- net N$11: track 48.9 -> 45.8 mm
- net 3.3V: track 241.7 -> 244.0 mm, vias 9 -> 7
- net N$17: track 48.6 -> 46.5 mm
- net N$18: track 5.25 -> 6.31 mm
Other:
- outline, holes or cut-outs redrawn

Commit message: adding panel
Parts:
- turned D3 to 180 degrees
- turned D4 to 180 degrees
Routing:
- net N$17: track 46.5 -> 44.4 mm
- net N$11: track 45.8 -> 44.8 mm
- net N$18: track 6.31 -> 5.25 mm
- net N$12: track 5.25 -> 5.96 mm
Other:
- outline, holes or cut-outs redrawn
- board text added: "Route Out"
