File: Production/Qwiic Solid State Relay-Panel.brd (EAGLE design)
At the start: 90.2 x 67.3 mm, 73 parts, among them J2 Qwiic Right Angle, J3 Qwiic Right Angle, J9 AVR_SPI_PROG_3X2TESTPOINTS, K1 25A Solid State Relay, K2 25A Solid State Relay, Q1 600mA/40V, Q2 600mA/40V, U4 ATTINY84-ARDUINO

Commit message: adding panel
Parts:
- removed FRAME1: FRAME-LETTER, SparkFun-Aesthetics:CREATIVE_COMMONS
- added ADR1, ADR2, ADR3, PWR1, PWR2, PWR3: JUMPER-SMT_2_NC_TRACE_SILK, SparkFun-Jumpers:SMT-JUMPER_2_NC_TRACE_SILK
- added C1, C2, C3: 0.1uF, SparkFun-Capacitors:0603
- added D10, D13, D16, D18, D5, D7: BLUE, SparkFun-LED:LED-0603
- added D12, D17, D6: RED, SparkFun-LED:LED-0603
- added D14, D15, D19, D20, D8, D9: (no value), SparkFun-LED:LED_5MM
- added E$1, E$2, E$3, E$4: (no value), SparkFun-Aesthetics:FIDUCIAL-1X2
- added E$5: (no value), SparkFun-Retired:FIDUCIAL-1.5X3
- added FD10, FD11, FD12, FD13, FD14, FD15, FD16, FD5, FD6, FD7, FD8, FD9: FIDUCIAL1X2, SparkFun-Aesthetics:FIDUCIAL-1X2
- added I2C1, I2C2, I2C3: JUMPER-SMT_3_2-NC_TRACE_SILK, SparkFun-Jumpers:SMT-JUMPER_3_2-NC_TRACE_SILK
- added J10, J16, J17, J23, J24, J8: Qwiic Right Angle, SparkFun-Connectors:JST04_1MM_RA
- added J11, J18, J25: AVR_SPI_PROG_3X2TESTPOINTS, SparkFun-Connectors:2X3_TEST_POINTS
- added J12, J13, J19, J20, J26, J27: (no value), SparkFun-Connectors:1X02_6.35_SCREWTERM
- added J14, J21, J28: (no value), SparkFun-Connectors:1X01_NO_SILK
- added J15, J22, J7: (no value), SparkFun-Connectors:1X04_NO_SILK
- added JP11, JP12, JP13, JP14, JP15, JP16, JP17, JP18, JP19, JP20, JP21, JP22, JP23, JP24, JP25, JP26, JP27, JP28, JP29, JP30, JP31, JP32, JP33, JP34, JP35, JP36, JP9: STAND-OFF, SparkFun-Hardware:STAND-OFF
- added K3, K4, K5, K6, K7, K8: 25A Solid State Relay, SparkFun-DiscreteSemi:PTH_SOLIDSTATERELAY
- added LOGO10, LOGO14, LOGO6: SFE_LOGO_NAME_FLAME.2_INCH, SparkFun-Aesthetics:SFE_LOGO_NAME_FLAME_.2
- added LOGO11, LOGO15, LOGO7: SFE_LOGO_NAME_FLAME.3_INCH, SparkFun-Aesthetics:SFE_LOGO_NAME_FLAME_.3
- added LOGO12, LOGO16, LOGO8: QWIIC_LOGO_5MM, SparkFun-Aesthetics:QWIIC_5MM
- added LOGO13, LOGO5, LOGO9: OSHW-LOGOS, SparkFun-Aesthetics:OSHW-LOGO-S
- added Q3, Q4, Q5, Q6, Q7, Q8: 600mA/40V, SparkFun-DiscreteSemi:SOT23-3
- added R10, R16, R18, R20, R23, R24, R25, R26, R29, R30, R32, R35, R36, R37, R38, R41, R42, R44, R47, R48, R9: 1k, SparkFun-Resistors:0603
- added R12, R21, R22, R27, R33, R34, R39, R45, R46: 4.7k, SparkFun-Resistors:0603
- added R13, R19, R28, R31, R40, R43: 47, SparkFun-Resistors:0603
- added U$22, U$26, U$46, U$48, U$68, U$70: (no value), buzzard_labels (11):22
- added U$25, U$4, U$45, U$47, U$67, U$69: (no value), buzzard_labels (11):11
- added U$27, U$28, U$49, U$50, U$71, U$72: (no value), SparkFun-Buzzard:GND_P
- added U$29, U$51, U$73: (no value), SparkFun-Buzzard:I2C
- added U$30, U$31, U$52, U$53, U$74, U$75: (no value), SparkFun-Buzzard:3V3_P
- added U$32, U$33, U$54, U$55, U$76, U$77: (no value), SparkFun-Buzzard:SCL_IO
- added U$34, U$35, U$56, U$57, U$78, U$79: (no value), SparkFun-Buzzard:SDA_IO
- added U$36, U$58, U$80: (no value), buzzard_labels (13):ADR3
- added U$37, U$59, U$81: (no value), SparkFun-Buzzard:PWR_TO
- added U$38, U$60, U$82: (no value), buzzard_labels (16):DUAL_SOLID0
- added U$39, U$61, U$83: (no value), buzzard_labels (16):STATE_RELAY1
- added U$40, U$41, U$62, U$63, U$84, U$85: (no value), buzzard_labels (19):HIGH_VOLTAGE0
- added U$42, U$43, U$64, U$65, U$86, U$87: (no value), SparkFun-Buzzard:RST_I
- added U$44, U$66, U$88: (no value), buzzard_labels (20):DUAL_SOLID_STATE_RELAY0
- added U1, U2, U3: ATTINY84-ARDUINO, SparkFun-IC-Microcontroller:SO14
Connections:
- new net !RESET1: J11.5, J14.1, R12.2, U1.4
- new net !RESET2: J18.5, J21.1, R27.2, U2.4
- new net !RESET3: J25.5, J28.1, R39.2, U3.4
- new net 3.3V1: C1.1, D6.A, I2C1.2, J10.2, J11.2, J7.3, J8.2, K3.3, K4.3, R12.1, R18.2, R23.2, R24.2, R9.2, U1.1
- new net 3.3V2: C2.1, D12.A, I2C2.2, J15.3, J16.2, J17.2, J18.2, K5.3, K6.3, R25.2, R27.1, R30.2, R35.2, R36.2, U2.1
- new net 3.3V3: C3.1, D17.A, I2C3.2, J22.3, J23.2, J24.2, J25.2, K7.3, K8.3, R37.2, R39.1, R42.2, R47.2, R48.2, U3.1
- new net ADDR_JUMP1: ADR1.1, U1.6
- new net ADDR_JUMP2: ADR2.1, U2.6
- new net ADDR_JUMP3: ADR3.1, U3.6
- new net GND1: ADR1.2, C1.2, J10.1, J11.6, J7.4, J8.1, PWR1.1, Q3.2, Q4.2, U1.14
- new net GND2: ADR2.2, C2.2, J15.4, J16.1, J17.1, J18.6, PWR2.1, Q5.2, Q6.2, U2.14
- new net GND3: ADR3.2, C3.2, J22.4, J23.1, J24.1, J25.6, PWR3.1, Q7.2, Q8.2, U3.14
- new net MISO1: J11.1, U1.8
- new net MISO2: J18.1, U2.8
- new net MISO3: J25.1, U3.8
- new net N$1: D6.C, R10.1
- new net N$19: K3.4, R13.2
- new net N$2: PWR1.2, R10.2
- new net N$20: D5.A, R9.1
- new net N$21: K4.4, R19.2
- new net N$22: D7.A, R18.1
- new net N$23: I2C1.3, R22.1
- new net N$24: I2C1.1, R21.1
- new net N$25: J12.P1, K3.2
- new net N$26: J12.P2, K3.1
- new net N$27: J13.P1, K4.2
- new net N$28: J13.P2, K4.1
- new net N$29: D5.C, D8.K, Q3.3, R13.1
- new net N$30: D8.A, R23.1
- new net N$31: D7.C, D9.K, Q4.3, R19.1
- new net N$32: D9.A, R24.1
- new net N$33: D12.C, R26.1
- new net N$34: PWR2.2, R26.2
- new net N$35: K5.4, R28.2
- new net N$36: D10.A, R25.1
- new net N$37: K6.4, R31.2
- new net N$38: D13.A, R30.1
- new net N$39: I2C2.3, R34.1
- new net N$40: I2C2.1, R33.1
- new net N$41: J19.P1, K5.2
- new net N$42: J19.P2, K5.1
- new net N$43: J20.P1, K6.2
- new net N$44: J20.P2, K6.1
- new net N$45: D10.C, D14.K, Q5.3, R28.1
- new net N$46: D14.A, R35.1
- new net N$47: D13.C, D15.K, Q6.3, R31.1
- new net N$48: D15.A, R36.1
- new net N$49: D17.C, R38.1
- new net N$50: PWR3.2, R38.2
- new net N$51: K7.4, R40.2
- new net N$52: D16.A, R37.1
- new net N$53: K8.4, R43.2
- new net N$54: D18.A, R42.1
- new net N$55: I2C3.3, R46.1
- new net N$56: I2C3.1, R45.1
- new net N$57: J26.P1, K7.2
- new net N$58: J26.P2, K7.1
- new net N$59: J27.P1, K8.2
- new net N$60: J27.P2, K8.1
- new net N$61: D16.C, D19.K, Q7.3, R40.1
- new net N$62: D19.A, R47.1
- new net N$63: D18.C, D20.K, Q8.3, R43.1
- new net N$64: D20.A, R48.1
- new net OPTO_3: Q3.1, R16.1
- new net OPTO_4: Q4.1, R20.1
- new net OPTO_5: Q5.1, R29.1
- new net OPTO_6: Q6.1, R32.1
- new net OPTO_7: Q7.1, R41.1
- new net OPTO_8: Q8.1, R44.1
- new net RELAY_CTRL3: R16.2, U1.10
- new net RELAY_CTRL4: R20.2, U1.11
- new net RELAY_CTRL5: R29.2, U2.10
- new net RELAY_CTRL6: R32.2, U2.11
- new net RELAY_CTRL7: R41.2, U3.10
- new net RELAY_CTRL8: R44.2, U3.11
- new net SCL/SCK1: J10.4, J11.3, J7.1, J8.4, R22.2, U1.9
- new net SCL/SCK2: J15.1, J16.4, J17.4, J18.3, R34.2, U2.9
- new net SCL/SCK3: J22.1, J23.4, J24.4, J25.3, R46.2, U3.9
- new net SDA/MOSI1: J10.3, J11.4, J7.2, J8.3, R21.2, U1.7
- new net SDA/MOSI2: J15.2, J16.3, J17.3, J18.4, R33.2, U2.7
- new net SDA/MOSI3: J22.2, J23.3, J24.3, J25.4, R45.2, U3.7
Routing:
- net 3.3V2: track 0.00 -> 241.7 mm, vias 0 -> 9
- net 3.3V1: track 0.00 -> 241.7 mm, vias 0 -> 9
- net 3.3V3: track 0.00 -> 241.7 mm, vias 0 -> 9
- net SDA/MOSI3: track 0.00 -> 107.0 mm, vias 0 -> 2
- net SDA/MOSI1: track 0.00 -> 107.0 mm, vias 0 -> 2
- net SDA/MOSI2: track 0.00 -> 107.0 mm, vias 0 -> 2
- net SCL/SCK3: track 0.00 -> 97.7 mm, vias 0 -> 2
- net SCL/SCK2: track 0.00 -> 97.7 mm, vias 0 -> 2
- net SCL/SCK1: track 0.00 -> 97.7 mm, vias 0 -> 2
- net !RESET1: track 0.00 -> 52.4 mm, vias 0 -> 1
- net !RESET3: track 0.00 -> 52.4 mm, vias 0 -> 1
- net !RESET2: track 0.00 -> 52.4 mm, vias 0 -> 1
- net N$29: track 0.00 -> 48.9 mm
- net N$61: track 0.00 -> 48.9 mm
- net N$45: track 0.00 -> 48.9 mm
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- added copper zone on layer 1, net GND1
- added copper zone on layer 16, net GND1
- added copper zone on layer 1, net GND2
- added copper zone on layer 16, net GND2
- added copper zone on layer 1, net GND3
- added copper zone on layer 16, net GND3
- added copper zone on layer 1, net N$25
- added copper zone on layer 16, net N$25
- added copper zone on layer 1, net N$26
- added copper zone on layer 16, net N$26
- added copper zone on layer 1, net N$27
- added copper zone on layer 16, net N$27
- added copper zone on layer 1, net N$28
- added copper zone on layer 16, net N$28
- added copper zone on layer 1, net N$41
- added copper zone on layer 16, net N$41
- added copper zone on layer 1, net N$42
- added copper zone on layer 16, net N$42
- added copper zone on layer 1, net N$43
- added copper zone on layer 16, net N$43
- added copper zone on layer 1, net N$44
- added copper zone on layer 16, net N$44
- added copper zone on layer 1, net N$57
- added copper zone on layer 16, net N$57
- added copper zone on layer 1, net N$58
- added copper zone on layer 16, net N$58
- added copper zone on layer 1, net N$59
- added copper zone on layer 16, net N$59
- added copper zone on layer 1, net N$60
- added copper zone on layer 16, net N$60
Other:
- board size 90.2 x 67.3 mm -> 200.9 x 155.2 mm
- board text added: "v-score"
- board text removed: "Andy England"

Commit message: adding panel
Parts:
- moved J12 17.8 mm to (104.6, 59.1), turned to 180 degrees
- moved J19 17.8 mm to (14.0, 126.9), turned to 180 degrees
- moved J20 17.8 mm to (58.4, 126.9), turned to 180 degrees
- moved J26 17.8 mm to (104.6, 126.9), turned to 180 degrees
- moved J4 17.8 mm to (14.0, 59.1), turned to 180 degrees
- moved J5 17.8 mm to (58.4, 59.1), turned to 180 degrees
- moved J13 17.8 mm to (149.1, 59.1), turned to 180 degrees
- moved J27 17.8 mm to (149.1, 126.9), turned to 180 degrees
- moved U$40 17.8 mm to (110.9, 62.2)
- moved U$84 17.8 mm to (110.9, 130.0)
- moved U$41 17.8 mm to (155.3, 62.2)
- moved U$63 17.8 mm to (64.6, 130.0)
- moved U$8 17.8 mm to (64.6, 62.2)
- moved U$85 17.8 mm to (155.3, 130.0)
- moved U$62 17.8 mm to (20.2, 130.0)
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Routing:
- net N$53: track 25.7 -> 19.9 mm
- net N$21: track 25.7 -> 19.9 mm
- net N$37: track 25.7 -> 19.9 mm
- net N$3: track 25.7 -> 19.9 mm
- net N$63: track 48.6 -> 44.4 mm
- net N$47: track 48.6 -> 44.4 mm
- net N$31: track 48.6 -> 44.4 mm
- net N$17: track 48.6 -> 44.4 mm
- net N$29: track 48.9 -> 44.8 mm
- net N$11: track 48.9 -> 44.8 mm
- net N$61: track 48.9 -> 44.8 mm
- net N$45: track 48.9 -> 44.8 mm
- net N$51: track 21.9 -> 18.5 mm
- net N$35: track 21.9 -> 18.5 mm
- net N$19: track 21.9 -> 18.5 mm
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Other:
- outline, holes or cut-outs redrawn
- board text added: "Route Out"
